Commit message: yeni duzenlemeler yaptim

File: src/my_robot_description/urdf/my_robot.urdf.xacro (robot description, xacro)
@@ -178,14 +178,6 @@
         <axis xyz="0 1 0"/>
     </joint>
-        <!-- Kamera gövdesi -->
+    <!-- Kamera gövdesi -->
     <link name="camera_link">
-        <visual>
-            <geometry>
-                <box size="0.08 0.12 0.08"/>
-            </geometry>
-            <material name="camera_black">
-                <color rgba="0.05 0.05 0.05 1.0"/>
-            </material>
-        </visual>
         <collision>
             <geometry>
@@ -224,5 +216,5 @@
             <always_on>true</always_on>
             <update_rate>30.0</update_rate>
-            <visualize>true</visualize>
+            <visualize>false</visualize>
             <camera name="front_camera">
                 <horizontal_fov>1.396</horizontal_fov>
